Commit message: changes to commit: 	add: launch file to bring up gazebo j2s7s300 robot in gazebo with rviz/moveit 	edit: robot description/launch files with new macro file destinations 	      planning_context condition for workstation/no workstation in robot_description param

File: kinova_description/urdf/j2s7s300_standalone.xacro (robot description, xacro)
@@ -2,31 +2,24 @@
 <!-- j2s7s300 refers to jaco v2 7DOF spherical 3fingers -->
 <robot xmlns:xi="http://www.w3.org/2001/XInclude"
-	xmlns:gazebo="http://playerstage.sourceforge.net/gazebo/xmlschema/#gz"
-    xmlns:model="http://playerstage.sourceforge.net/gazebo/xmlschema/#model"
-	xmlns:sensor="http://playerstage.sourceforge.net/gazebo/xmlschema/#sensor"
-	xmlns:body="http://playerstage.sourceforge.net/gazebo/xmlschema/#body"
-    xmlns:geom="http://playerstage.sourceforge.net/gazebo/xmlschema/#geom"
-    xmlns:joint="http://playerstage.sourceforge.net/gazebo/xmlschema/#joint"
-	xmlns:controller="http://playerstage.sourceforge.net/gazebo/xmlschema/#controller"
-	xmlns:interface="http://playerstage.sourceforge.net/gazebo/xmlschema/#interface"
-	xmlns:rendering="http://playerstage.sourceforge.net/gazebo/xmlschema/#rendering"
-    xmlns:renderable="http://playerstage.sourceforge.net/gazebo/xmlschema/#renderable"
-    xmlns:physics="http://playerstage.sourceforge.net/gazebo/xmlschema/#physics"
-	xmlns:xacro="http://www.ros.org/wiki/xacro" name="j2s7s300">
+  xmlns:gazebo="http://playerstage.sourceforge.net/gazebo/xmlschema/#gz"
+  xmlns:model="http://playerstage.sourceforge.net/gazebo/xmlschema/#model"
+  xmlns:sensor="http://playerstage.sourceforge.net/gazebo/xmlschema/#sensor"
+  xmlns:body="http://playerstage.sourceforge.net/gazebo/xmlschema/#body"
+  xmlns:geom="http://playerstage.sourceforge.net/gazebo/xmlschema/#geom"
+  xmlns:joint="http://playerstage.sourceforge.net/gazebo/xmlschema/#joint"
+  xmlns:controller="http://playerstage.sourceforge.net/gazebo/xmlschema/#controller"
+  xmlns:interface="http://playerstage.sourceforge.net/gazebo/xmlschema/#interface"
+  xmlns:rendering="http://playerstage.sourceforge.net/gazebo/xmlschema/#rendering"
+  xmlns:renderable="http://playerstage.sourceforge.net/gazebo/xmlschema/#renderable"
+  xmlns:physics="http://playerstage.sourceforge.net/gazebo/xmlschema/#physics"
+  xmlns:xacro="http://www.ros.org/wiki/xacro" name="j2s7s300">
   <xacro:include filename="$(find kinova_description)/urdf/j2s7s300.xacro"/>
-  <xacro:include filename="$(find uml_hri_nerve_pick_and_place)/urdf/workstation_model.urdf.xacro" />
-  <xacro:workstation prefix="table_"/>
+  <link name="root"/>
   <!-- for gazebo -->
   <link name="world"/>
-  <joint name="connect_world_and_table" type="fixed">
-    <child link="table_base_link" />
+  <joint name="connect_root_and_world" type="fixed">
+    <child link="root" />
     <parent link="world" />
-    <origin xyz="0.0 0.0 0.41" rpy="0.0 0.0 0.0" />
-  </joint>
-  <link name="root"/>
-  <joint name="connect_table_and_root" type="fixed">
-    <child link="root" />
-    <parent link="table_mounting_plate_link" />
-    <origin xyz="0.0 0.0 0.03625" rpy="0.0 0.0 ${-pi/2}" />
+    <origin xyz="0 0 0" rpy="0 0 0" />
   </joint>
   <xacro:property name="robot_root" value="root" />

File: kinova_description/urdf/j2s7s300_workstation.xacro (robot description, xacro)
@@ -15,5 +15,5 @@
 	xmlns:xacro="http://www.ros.org/wiki/xacro" name="j2s7s300">
   <xacro:include filename="$(find kinova_description)/urdf/j2s7s300.xacro"/>
-  <xacro:include filename="$(find uml_hri_nerve_pick_and_place)/urdf/workstation_model.urdf.xacro" />
+  <xacro:include filename="$(find uml_hri_nerve_armada_workstation)/workstation_description/workstation_model.urdf.xacro" />
   <xacro:workstation prefix="table_"/>
   <!-- for gazebo -->
