Commit message: Changes to commit: create more universal launch file for workstation sim configuration with support for multiple robots     add: description for robot and workstation for each robot with a moveit config, gazebo grasping plugin support for each robot with a moveit config     modify: gazebo_demo and planning_context launch files for each robot with a moveit_config; add workstation_sim arguments to allow for more seamless launching while preserving existing launch files and commands     remove: j2s7s300 specific workstation_sim related launch files from j2s7s300 moveit_config package

File: kinova_description/urdf/j2n6s300.xacro (robot description, xacro)
@@ -16,4 +16,5 @@
     <xacro:include filename="$(find kinova_description)/urdf/kinova_common.xacro" />
     <xacro:include filename="$(find kinova_description)/urdf/kinova_finger_set.xacro" />
+    <xacro:include filename="$(find kinova_description)/urdf/three_finger_gripping_gazebo.xacro" />
     <!-- Import all Gazebo-customization elements -->
     <xacro:include filename="$(find kinova_description)/urdf/kinova.gazebo" />
@@ -120,5 +121,6 @@
         <xacro:kinova_virtual_link link_name="${prefix}_end_effector"/>
         <xacro:kinova_virtual_joint joint_name="${prefix}_joint_end_effector" type="${joint_end_effector_type}" parent="${prefix}_link_6" child="${prefix}_end_effector" joint_axis_xyz="${joint_end_effector_axis_xyz}" joint_origin_xyz="${joint_end_effector_origin_xyz}" joint_origin_rpy="${joint_end_effector_origin_rpy}" joint_lower_limit="0" joint_upper_limit="0"/>
-    <xacro:kinova_3fingers link_hand="${prefix}_link_6" prefix="${prefix}_"/>
+        <xacro:kinova_3fingers link_hand="${prefix}_link_6" prefix="${prefix}_"/>
+        <xacro:three_finger_gripping_gazebo robot="${prefix}" DoF="6"/>
     </xacro:macro>
 </root>

File: kinova_description/urdf/j2s6s300.xacro (robot description, xacro)
@@ -16,4 +16,5 @@
     <xacro:include filename="$(find kinova_description)/urdf/kinova_common.xacro" />
     <xacro:include filename="$(find kinova_description)/urdf/kinova_finger_set.xacro" />
+    <xacro:include filename="$(find kinova_description)/urdf/three_finger_gripping_gazebo.xacro" />
     <!-- Import all Gazebo-customization elements -->
     <xacro:include filename="$(find kinova_description)/urdf/kinova.gazebo" />
@@ -120,5 +121,6 @@
         <xacro:kinova_virtual_link link_name="${prefix}_end_effector"/>
         <xacro:kinova_virtual_joint joint_name="${prefix}_joint_end_effector" type="${joint_end_effector_type}" parent="${prefix}_link_6" child="${prefix}_end_effector" joint_axis_xyz="${joint_end_effector_axis_xyz}" joint_origin_xyz="${joint_end_effector_origin_xyz}" joint_origin_rpy="${joint_end_effector_origin_rpy}" joint_lower_limit="0" joint_upper_limit="0"/>
-    <xacro:kinova_3fingers link_hand="${prefix}_link_6" prefix="${prefix}_"/>
+        <xacro:kinova_3fingers link_hand="${prefix}_link_6" prefix="${prefix}_"/>
+        <xacro:three_finger_gripping_gazebo robot="${prefix}" DoF="6"/>
     </xacro:macro>
 </robot>

File: kinova_description/urdf/j2s7s300.xacro (robot description, xacro)
@@ -135,5 +135,5 @@
         <xacro:kinova_virtual_joint joint_name="${prefix}_joint_end_effector" type="${joint_end_effector_type}" parent="${prefix}_link_7" child="${prefix}_end_effector" joint_axis_xyz="${joint_end_effector_axis_xyz}" joint_origin_xyz="${joint_end_effector_origin_xyz}" joint_origin_rpy="${joint_end_effector_origin_rpy}" joint_lower_limit="0" joint_upper_limit="0"/>
         <xacro:kinova_3fingers link_hand="${prefix}_link_7" prefix="${prefix}_"/>
-        <xacro:three_finger_gripping_gazebo robot="${prefix}" />
+        <xacro:three_finger_gripping_gazebo robot="${prefix}" DoF="7"/>
     </xacro:macro>
 </root>

File: kinova_description/urdf/j2s7s300_workstation.xacro (robot description, xacro)
@@ -17,5 +17,4 @@
   <xacro:include filename="$(find uml_hri_nerve_armada_workstation)/workstation_description/workstation_model.urdf.xacro" />
   <xacro:workstation prefix="table_"/>
-  <!-- for gazebo -->
   <link name="world"/>
   <joint name="connect_world_and_table" type="fixed">

File: kinova_description/urdf/m1n6s300.xacro (robot description, xacro)
@@ -16,4 +16,5 @@
     <xacro:include filename="$(find kinova_description)/urdf/kinova_common.xacro" />
     <xacro:include filename="$(find kinova_description)/urdf/kinova_finger_set.xacro" />
+    <xacro:include filename="$(find kinova_description)/urdf/three_finger_gripping_gazebo.xacro" />
     <!-- Import all Gazebo-customization elements -->
     <xacro:include filename="$(find kinova_description)/urdf/kinova.gazebo" />
@@ -120,5 +121,6 @@
         <xacro:kinova_virtual_link link_name="${prefix}_end_effector"/>
         <xacro:kinova_virtual_joint joint_name="${prefix}_joint_end_effector" type="${joint_end_effector_type}" parent="${prefix}_link_6" child="${prefix}_end_effector" joint_axis_xyz="${joint_end_effector_axis_xyz}" joint_origin_xyz="${joint_end_effector_origin_xyz}" joint_origin_rpy="${joint_end_effector_origin_rpy}" joint_lower_limit="0" joint_upper_limit="0"/>
-    <xacro:kinova_3fingers link_hand="${prefix}_link_6" prefix="${prefix}_"/>
+        <xacro:kinova_3fingers link_hand="${prefix}_link_6" prefix="${prefix}_"/>
+        <xacro:three_finger_gripping_gazebo robot="${prefix}" DoF="6"/>
     </xacro:macro>
 </root>

File: kinova_description/urdf/three_finger_gripping_gazebo.xacro (robot description, xacro)
@@ -1,4 +1,3 @@
 <?xml version="1.0"?>
-<!-- j2s7s300 refers to jaco v2 7DOF spherical 3fingers -->
 <robot xmlns:xi="http://www.w3.org/2001/XInclude"
   xmlns:gazebo="http://playerstage.sourceforge.net/gazebo/xmlschema/#gz"
@@ -14,10 +13,10 @@
   xmlns:physics="http://playerstage.sourceforge.net/gazebo/xmlschema/#physics"
   xmlns:xacro="http://www.ros.org/wiki/xacro" name="j2s7s300">
-  <xacro:macro name="three_finger_gripping_gazebo" params="robot">
+  <xacro:macro name="three_finger_gripping_gazebo" params="robot DoF">
     <gazebo>
        <plugin name="gazebo_grasp_fix" filename="libgazebo_grasp_fix.so">
          <arm>
            <arm_name>${robot}</arm_name>
-           <palm_link>${robot}_link_7</palm_link>
+           <palm_link>${robot}_link_${DoF}</palm_link>
            <gripper_link>${robot}_link_finger_1</gripper_link>
            <gripper_link>${robot}_link_finger_tip_1</gripper_link>
