Commit message: add: real jaco2 bringup with actual realsense2 camera; update robot description - rotate robot into place; add static transform publisher for camera frame

File: kinova_description/urdf/j2s7s300_workstation.xacro (robot description, xacro)
@@ -27,5 +27,5 @@
     <child link="root" />
     <parent link="table_mounting_plate_link" />
-    <origin xyz="0.0 0.0 0.03625" rpy="0.0 0.0 ${-pi/2}" />
+    <origin xyz="0.0 0.0 0.03625" rpy="0.0 0.0 ${pi}" />
   </joint>
   <xacro:property name="robot_root" value="root" />
